File: Schematic/EAGLE/MCUTNC/MCUTNC.sch (EAGLE design)
At the start: 7 parts, among them Q1 MPSA56-TO92, U1 NUCLEO-F446RE

Commit message: dumb temp files
Parts:
- added J1: AUDIO_JACK_TRRSSMD_RA, SparkFun-Connectors:AUDIO_JACK_TRRSSMD_RA
Connections:
- new net AUIDO_0V5_OUT: J1.RING2
- net AUDIO_IN: now also J1.TIP
- net GND: now also J1.EARTH
- net PTT_15V: now also J1.RING1
Other:
- moved on the sheet: C1, C2, Q1, R1, R2, R3, U1G$4, U1G$5
